File: KiCAD/MVX_Audio_Separator/MVX_Audio_Separator.kicad_pcb (KiCad board)
At the start: 2 copper layers, 30.9 x 26.9 mm, 4 parts, among them J1 3.5mm_vertical, P1 VGA_Female, P2 VGA_Male

Commit message: Update PCB
Other:
- board size 30.9 x 26.9 mm -> 30.8 x 26.8 mm

Commit message: Update PCB
Parts:
- moved J1 5.00 mm to (138.3, 101.2)
Routing:
- net /Audio_R: track 9.47 -> 14.5 mm
- net /Red: track 18.1 -> 22.7 mm
- net /Green: track 16.5 -> 20.6 mm
- net /HSYNC: track 41.6 -> 39.6 mm
- net /Blue: track 12.9 -> 14.1 mm
- net /Audio_L: track 22.7 -> 21.8 mm
- net GND: vias 20 -> 16
